File: GettingToBlinky5.0.kicad_pcb (KiCad board)
At the start: 2 copper layers, 7 parts, among them U1 7555

Commit message: Finishing The Layout
Parts:
- BT1: moved to B.Cu
- moved R1 24.3 mm to (152.5, 92.5), turned to -90 degrees
- moved R2 23.7 mm to (152.5, 96.5), turned to -90 degrees
- moved R3 19.0 mm to (138.5, 95.5), turned to -90 degrees
- moved C1 18.6 mm to (138.5, 91.5), turned to 90 degrees
- moved U1 16.7 mm to (145.5, 94.0)
- moved D1 14.3 mm to (138.5, 99.5), turned to 90 degrees
- moved BT1 2.18 mm to (145.5, 94.0), turned to 180 degrees
Connections:
- net Net-(BT1-+) renamed /VDD
- net Net-(U1-DIS) renamed /DIS
- net Net-(U1-THR) renamed /THR
Routing:
- net /THR: track 0.00 -> 16.1 mm
- net /VDD: track 0.00 -> 15.3 mm, vias 0 -> 2
- net GND: track 0.00 -> 9.60 mm, vias 0 -> 2
- net /DIS: track 0.00 -> 6.58 mm
- net Net-(U1-OUT): track 0.00 -> 4.58 mm
- net Net-(D1-A): track 0.00 -> 2.00 mm
- added copper zone on F.Cu, net /VDD
- added copper zone on B.Cu, net GND
Other:
- board outline added: 33 x 30.1 mm

Commit message: Output Files For Manufacturing
Other:
- board text added: "Hello Blinky"
Changed lines of the file:
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@@
 			(outputformat 1)
 			(mirror no)
-			(drillshape 1)
+			(drillshape 0)
 			(scaleselection 1)
-			(outputdirectory "")
+			(outputdirectory "Gerber/")
 		)
 	)
@@
 		(tags "resistor handsolder")
 		(property "Reference" "R2"
-			(at 0 -1.65 90)
-			(layer "F.SilkS")
-			(effects
-				(font
-					(size 1 1)
-					(thickness 0.15)
+			(at 0 -2 90)
+			(unlocked yes)
+			(layer "F.SilkS")
+			(effects
+				(font
+					(size 1.2 1.2)
+					(thickness 0.1)
 				)
 			)
@@
 			(at 0 1.65 90)
 			(layer "F.Fab")
+			(hide yes)
 			(effects
 				(font
@@
 		(fp_text user "${REFERENCE}"
 			(at 0 0 90)
-			(layer "F.Fab")
-			(effects
-				(font
-					(size 0.5 0.5)
-					(thickness 0.08)
+			(unlocked yes)
+			(layer "F.Fab")
+			(effects
+				(font
+					(size 1 1)
+					(thickness 0.15)
 				)
 			)
@@
 		(tags "resistor handsolder")
 		(property "Reference" "R3"
-			(at 0 -1.65 90)
-			(layer "F.SilkS")
-			(effects
-				(font
-					(size 1 1)
-					(thickness 0.15)
+			(at 0 2 90)
+			(unlocked yes)
+			(layer "F.SilkS")
+			(effects
+				(font
+					(size 1.2 1.2)
+					(thickness 0.1)
 				)
 			)
@@
 			(at 0 1.65 90)
 			(layer "F.Fab")
+			(hide yes)
 			(effects
 				(font
@@
 		(fp_text user "${REFERENCE}"
 			(at 0 0 90)
-			(layer "F.Fab")
-			(effects
-				(font
-					(size 0.5 0.5)
-					(thickness 0.08)
+			(unlocked yes)
+			(layer "F.Fab")
+			(effects
+				(font
+					(size 1 1)
+					(thickness 0.15)
 				)
 			)
@@
 		(tags "SOIC SO")
 		(property "Reference" "U1"
-			(at 0 -3.4 0)
-			(layer "F.SilkS")
-			(effects
-				(font
-					(size 1 1)
-					(thickness 0.15)
+			(at 0 -3.75 0)
+			(unlocked yes)
+			(layer "F.SilkS")
+			(effects
+				(font
+					(size 1.2 1.2)
+					(thickness 0.1)
 				)
 			)
@@
 			(at 0 3.4 0)
 			(layer "F.Fab")
+			(hide yes)
 			(effects
 				(font
@@
 		(fp_text user "${REFERENCE}"
 			(at 0 0 90)
+			(unlocked yes)
 			(layer "F.Fab")
 			(effects
@@
 		(tags "LED handsolder")
 		(property "Reference" "D1"
-			(at 0 -1.65 90)
-			(layer "F.SilkS")
-			(effects
-				(font
-					(size 1 1)
-					(thickness 0.15)
+			(at 0 -2 90)
+			(unlocked yes)
+			(layer "F.SilkS")
+			(effects
+				(font
+					(size 1.2 1.2)
+					(thickness 0.1)
 				)
 			)
@@
 			(at 0 1.65 90)
 			(layer "F.Fab")
+			(hide yes)
 			(effects
 				(font
@@
 		(fp_text user "${REFERENCE}"
 			(at 0 0 90)
-			(layer "F.Fab")
-			(effects
-				(font
-					(size 0.5 0.5)
-					(thickness 0.08)
+			(unlocked yes)
+			(layer "F.Fab")
+			(effects
+				(font
+					(size 1 1)
+					(thickness 0.15)
 				)
 			)
@@
 		(tags "capacitor handsolder")
 		(property "Reference" "C1"
-			(at 0 -1.68 90)
-			(layer "F.SilkS")
-			(effects
-				(font
-					(size 1 1)
-					(thickness 0.15)
+			(at 0 -2 90)
+			(unlocked yes)
+			(layer "F.SilkS")
+			(effects
+				(font
+					(size 1.2 1.2)
+					(thickness 0.1)
 				)
 			)
@@
 			(at 0 1.68 90)
 			(layer "F.Fab")
+			(hide yes)
 			(effects
 				(font
@@
 		(fp_text user "${REFERENCE}"
 			(at 0 0 90)
-			(layer "F.Fab")
-			(effects
-				(font
-					(size 0.5 0.5)
-					(thickness 0.08)
+			(unlocked yes)
+			(layer "F.Fab")
+			(effects
+				(font
+					(size 1 1)
+					(thickness 0.15)
 				)
 			)
@@
 		(tags "resistor handsolder")
 		(property "Reference" "R1"
-			(at 0 -1.65 90)
-			(layer "F.SilkS")
-			(effects
-				(font
-					(size 1 1)
-					(thickness 0.15)
+			(at 0 -2 90)
+			(unlocked yes)
+			(layer "F.SilkS")
+			(effects
+				(font
+					(size 1.2 1.2)
+					(thickness 0.1)
 				)
 			)
@@
 			(at 0 1.65 90)
 			(layer "F.Fab")
+			(hide yes)
 			(effects
 				(font
@@
 		(fp_text user "${REFERENCE}"
 			(at 0 0 90)
-			(layer "F.Fab")
-			(effects
-				(font
-					(size 0.5 0.5)
-					(thickness 0.08)
+			(unlocked yes)
+			(layer "F.Fab")
+			(effects
+				(font
+					(size 1 1)
+					(thickness 0.15)
 				)
 			)
@@
 			(effects
 				(font
-					(size 1 1)
+					(size 1.2 1.2)
 					(thickness 0.1)
 				)
@@
 			(unlocked yes)
 			(layer "B.Fab")
+			(hide yes)
 			(effects
 				(font
@@
 		(layer "Edge.Cuts")
 	)
+	(gr_text "Hello Blinky"
+		(at 140.5 85.25 0)
+		(layer "F.SilkS")
+		(effects
+			(font
+				(size 1.2 1.2)
+				(thickness 0.1)
+			)
+			(justify left bottom)
+		)
+	)
 	(segment

Commit message: Create a pcb to send to jlcpcb
Parts:
- BT1: footprint GettingToBlinky5.0:S8211-46R -> Battery:BatteryHolder_Keystone_3034_1x20mm
Routing:
- net /VDD: track 15.3 -> 21.8 mm
- net GND: track 9.60 -> 14.6 mm
Other:
- board size 33 x 30.1 mm -> 25 x 25 mm
