File: GettingToBlinky5.0.kicad_sch (KiCad schematic)
At the start: 0 parts

Commit message: Schematic Symbol Creation
Parts:
- added U1: 7555, symbol GTB5:7555
Changed lines of the file:
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@@
 	(generator_version "9.0")
 	(paper "A4")
+	(symbol
+		(lib_id "GTB5:7555")
+		(at 140.97 101.6 0)
+		(unit 1)
+		(exclude_from_sim no)
+		(in_bom yes)
+		(on_board yes)
+		(dnp no)
+		(property "Reference" "U1"
+			(at 141.478 100.838 0)
+			(effects
+				(font
+					(size 1.27 1.27)
+				)
+			)
+		)
+		(property "Value" "7555"
+			(at 140.716 97.028 0)
+			(effects
+				(font
+					(size 1.27 1.27)
+				)
+			)
+		)
+		(property "Footprint" ""
+			(at 140.97 101.6 0)
+			(effects
+				(font
+					(size 1.27 1.27)
+				)
+				(hide yes)
+			)
+		)
+		(property "Datasheet" ""
+			(at 140.97 101.6 0)
+			(effects
+				(font
+					(size 1.27 1.27)
+				)
+				(hide yes)
+			)
+		)
+		(property "Description" ""
+			(at 140.97 101.6 0)
+			(effects
+				(font
+					(size 1.27 1.27)
+				)
+				(hide yes)
+			)
+		)
+		(pin "8"
+		)
+		(pin "1"
+		)
+		(pin "7"
+		)
+		(pin "4"
+		)
+		(pin "3"
+		)
+		(pin "5"
+		)
+		(pin "2"
+		)
+		(pin "6"
+		)
+		(instances
+			(project ""
+				(path "/5fa71722-745b-4065-a65e-13b56c379e5f"
+					(reference "U1")
+					(unit 1)
+				)
+			)
+		)
+	)
 	(sheet_instances
 		(path "/"

Commit message: Making The Schematic
Parts:
- added BT1: CR2032, symbol Device:Battery_Cell
- added C1: 1U, symbol Device:C
- added D1: LED, symbol Device:LED
- added R1, R3: 1K, symbol Device:R
- added R2: 470K, symbol Device:R
Connections:
- net GND: now reaches U1.1 (GND)
- net GND: now also BT1.2 (-), C1.2, D1.1 (K)
- net at U1.2 (~{TRIG}): now also U1.6 (THR), C1.1, R2.2
- net at U1.3 (OUT): now also R3.1
- net at U1.4 (~{RST}): now also U1.8 (VDD), BT1.1 (+), R1.1
- net at U1.7 (DIS): now also R1.2, R2.1
- new net: D1.2 (A), R3.2
- no-connect marks 0 -> 1

Commit message: Associating Symbol and Footprint
Parts:
- C1: footprint (none) -> Capacitor_SMD:C_0805_2012Metric_Pad1.18x1.45mm_HandSolder
- D1: footprint (none) -> LED_SMD:LED_0805_2012Metric_Pad1.15x1.40mm_HandSolder
- R1, R2, R3: footprint (none) -> Resistor_SMD:R_0805_2012Metric_Pad1.20x1.40mm_HandSolder
- U1: footprint (none) -> Package_SO:SOIC-8_3.9x4.9mm_P1.27mm
Changed lines of the file:
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@@
 			)
 		)
-		(property "Footprint" ""
+		(property "Footprint" "Resistor_SMD:R_0805_2012Metric_Pad1.20x1.40mm_HandSolder"
 			(at 104.902 101.6 90)
 			(effects
@@
 			)
 		)
-		(property "Footprint" ""
+		(property "Footprint" "Resistor_SMD:R_0805_2012Metric_Pad1.20x1.40mm_HandSolder"
 			(at 104.902 86.36 90)
 			(effects
@@
 			)
 		)
-		(property "Footprint" ""
+		(property "Footprint" "Resistor_SMD:R_0805_2012Metric_Pad1.20x1.40mm_HandSolder"
 			(at 167.132 115.57 90)
 			(effects
@@
 			)
 		)
-		(property "Footprint" ""
+		(property "Footprint" "Package_SO:SOIC-8_3.9x4.9mm_P1.27mm"
 			(at 140.97 101.6 0)
 			(effects
@@
 			)
 		)
-		(property "Footprint" ""
+		(property "Footprint" "LED_SMD:LED_0805_2012Metric_Pad1.15x1.40mm_HandSolder"
 			(at 168.91 129.54 0)
 			(effects
@@
 			)
 		)
-		(property "Footprint" ""
+		(property "Footprint" "Capacitor_SMD:C_0805_2012Metric_Pad1.18x1.45mm_HandSolder"
 			(at 107.6452 121.92 0)
 			(effects

Commit message: Creating A Custom Footprint
Parts:
- BT1: footprint (none) -> GettingToBlinky5.0:S8211-46R
Changed lines of the file:
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@@
 			)
 		)
-		(property "Footprint" ""
+		(property "Footprint" "GettingToBlinky5.0:S8211-46R"
 			(at 74.93 106.426 90)
 			(effects

Commit message: Finishing The Layout
Connections:
- net VDD: now reaches BT1.1 (+), R1.1, U1.4 (~{RST}), U1.8 (VDD)
- net DIS: now reaches R1.2, R2.1, U1.7 (DIS)
- net THR: now reaches C1.1, R2.2, U1.2 (~{TRIG}), U1.6 (THR)
Changed lines of the file:
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@@
+		)
+	)
+	(label "THR"
+		(at 115.57 107.95 0)
+		(effects
+			(font
+				(size 1.27 1.27)
+			)
+			(justify left bottom)
+		)
+	)
+	(label "VDD"
+		(at 124.46 67.31 0)
+		(effects
+			(font
+				(size 1.27 1.27)
+			)
+			(justify left bottom)
+		)
+	)
+	(label "DIS"
+		(at 118.11 93.98 0)
+		(effects
+			(font
+				(size 1.27 1.27)
+			)
+			(justify left bottom)
 		)
 	)

Commit message: Create a pcb to send to jlcpcb
Parts:
- BT1: footprint GettingToBlinky5.0:S8211-46R -> Battery:BatteryHolder_Keystone_3034_1x20mm
Changed lines of the file:
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@@
 			)
 		)
-		(property "Footprint" "GettingToBlinky5.0:S8211-46R"
+		(property "Footprint" "Battery:BatteryHolder_Keystone_3034_1x20mm"
 			(at 74.93 106.426 90)
 			(effects
